File: Elektronik/Transimpedanz/transimpendanzVerstaerker/transimpendanzVerstaerker.kicad_pcb (KiCad board)
At the start: 2 copper layers, 5 parts, among them J1 con1, U1 LM358

Commit message: finished test pcb layout
Parts:
- moved D1 4.02 mm to (130.8, 92.7)
- moved U1 2.84 mm to (141.0, 90.2)
Routing:
- net Net-(D1-Pad2): track 54.1 -> 64.0 mm
- net Net-(C1-Pad2): track 30.5 -> 37.4 mm
- net Net-(C1-Pad1): track 25.6 -> 28.7 mm
- net Net-(J1-Pad3): track 8.03 -> 9.30 mm
Other:
- board outline added: 29.2 x 26.7 mm
