File: Elektronik/NotLoesung/sensorBoard/sensorBoard.sch (KiCad schematic (older format))
At the start: 46 parts

Commit message: Schaltplan fertig
Parts:
- added J1: Conn_01x04_Male, symbol Connector:Conn_01x04_Male
- gave numbers to parts that had none: 30
Connections:
- wire segments 215 -> 247
Other:
- note added: "0x48"
- note added: "0x49"
- note added: "0x4A"
- note added: "0x4B"
- note added: "Interrupt 1- 4"
